File: greenpill.kicad_pcb (KiCad board)
At the start: 2 copper layers, 52.8 x 19 mm, 35 parts, among them CN1 CON-USB_5P, J1 1x20_HDR, J2 1x20_HDR, J3 1X4_HDR, SW1 SW_Push_2P, U1 CAT6219, U2 STM32F103C8T, Y1 32.768k, Y2 8M

Commit message: Update silk, routing.
Parts:
- moved C9 0.13 mm to (151.4, 98.4)
Routing:
- net GND: track 143.7 -> 160.4 mm
Other:
- board text added: "0"
- board text added: "1"
- board text added: "PC13"
- board text added: "PWR"
